Commit message: add room1

File: open_manipulator_with_tb3_description/urdf/open_manipulator_with_tb3.gazebo.xacro (robot description, xacro)
@@ -12,5 +12,5 @@
     <maxVel>1.0</maxVel>
     <minDepth>0.001</minDepth>
-    <material>Gazebo/DarkGrey</material>
+    <material>Gazebo/Gold</material>
   </gazebo>
   <!-- Link2 -->
@@ -22,5 +22,5 @@
     <maxVel>1.0</maxVel>
     <minDepth>0.001</minDepth>
-    <material>Gazebo/DarkGrey</material>
+    <material>Gazebo/Gold</material>
   </gazebo>
   <!-- Link3 -->
@@ -32,5 +32,5 @@
     <maxVel>1.0</maxVel>
     <minDepth>0.001</minDepth>
-    <material>Gazebo/DarkGrey</material>
+    <material>Gazebo/Gold</material>
   </gazebo>
   <!-- Link4 -->
@@ -42,5 +42,5 @@
     <maxVel>1.0</maxVel>
     <minDepth>0.001</minDepth>
-    <material>Gazebo/DarkGrey</material>
+    <material>Gazebo/Gold</material>
   </gazebo>
   <!-- Link5 -->
@@ -52,5 +52,5 @@
     <maxVel>1.0</maxVel>
     <minDepth>0.001</minDepth>
-    <material>Gazebo/DarkGrey</material>
+    <material>Gazebo/Gold</material>
   </gazebo>
   <!-- grip_link -->
@@ -62,5 +62,5 @@
     <maxVel>1.0</maxVel>
     <minDepth>0.001</minDepth>
-    <material>Gazebo/DarkGrey</material>
+    <material>Gazebo/Gold</material>
   </gazebo>
   <!-- grip_link_sub -->
@@ -72,5 +72,5 @@
     <maxVel>1.0</maxVel>
     <minDepth>0.001</minDepth>
-    <material>Gazebo/DarkGrey</material>
+    <material>Gazebo/Gold</material>
   </gazebo>
   <!-- ros_control plugin -->

File: open_manipulator_with_tb3_description/urdf/open_manipulator_with_tb3_waffle_pi.urdf.xacro (robot description, xacro)
@@ -20,4 +20,5 @@
       </geometry>
       <material name="grey"/>
+      <!--<material>Gazebo/Gold</material>-->
     </visual>
     <collision>
@@ -68,5 +69,6 @@
         <mesh filename="package://open_manipulator_with_tb3_description/meshes/chain_link2.stl" scale="0.001 0.001 0.001"/>
       </geometry>
-      <material name="grey"/>
+      <!--<material name="grey"/>-->
+      <material>Gazebo/Gold</material>
     </visual>
     <collision>
@@ -117,5 +119,6 @@
         <mesh filename="package://open_manipulator_with_tb3_description/meshes/chain_link3.stl" scale="0.001 0.001 0.001"/>
       </geometry>
-      <material name="grey"/>
+      <!--<material name="grey"/>-->
+      <material>Gazebo/Gold</material>
     </visual>
     <collision>
@@ -166,5 +169,6 @@
         <mesh filename="package://open_manipulator_with_tb3_description/meshes/chain_link4.stl" scale="0.001 0.001 0.001"/>
       </geometry>
-      <material name="grey"/>
+      <!--<material name="grey"/>-->
+      <material>Gazebo/Gold</material>
     </visual>
     <collision>
@@ -215,5 +219,6 @@
         <mesh filename="package://open_manipulator_with_tb3_description/meshes/chain_link5.stl" scale="0.001 0.001 0.001"/>
       </geometry>
-      <material name="grey"/>
+      <!--<material name="grey"/>-->
+      <material>Gazebo/Gold</material>
     </visual>
     <collision>
@@ -245,5 +250,6 @@
         <mesh filename="package://open_manipulator_with_tb3_description/meshes/chain_link_grip_l.stl" scale="0.001 0.001 0.001"/>
       </geometry>
-      <material name="grey"/>
+      <!--<material name="grey"/>-->
+      <material>Gazebo/Gold</material>
     </visual>
     <collision>
@@ -294,5 +300,6 @@
         <mesh filename="package://open_manipulator_with_tb3_description/meshes/chain_link_grip_r.stl" scale="0.001 0.001 0.001"/>
       </geometry>
-      <material name="grey"/>
+      <!--<material name="grey"/>-->
+      <material>Gazebo/Gold</material>
     </visual>
     <collision>

File: open_manipulator_with_tb3_description/urdf/turtlebot3_waffle2.gazebo.xacro (robot description, xacro)
@@ -5,5 +5,5 @@
   <xacro:arg name="imu_visual"    default="false"/>
   <gazebo reference="base_link">
-    <material>Gazebo/DarkGrey</material>
+    <material>Gazebo/Gold</material>
   </gazebo>
   <gazebo reference="wheel_left_link">
@@ -17,5 +17,5 @@
     <maxVel>0.1</maxVel>
     <fdir1>1 0 0</fdir1>
-    <material>Gazebo/FlatBlack</material>
+    <material>Gazebo/Black</material>
   </gazebo>
   <gazebo reference="wheel_right_link">
@@ -29,5 +29,5 @@
     <maxVel>0.1</maxVel>
     <fdir1>1 0 0</fdir1>
-    <material>Gazebo/FlatBlack</material>
+    <material>Gazebo/Black</material>
   </gazebo>
   <gazebo reference="caster_back_right_link">
@@ -38,5 +38,5 @@
     <minDepth>0.001</minDepth>
     <maxVel>1.0</maxVel>
-    <material>Gazebo/FlatBlack</material>
+    <material>Gazebo/Gold</material>
   </gazebo>
   <gazebo reference="caster_back_left_link">
@@ -47,5 +47,5 @@
     <minDepth>0.001</minDepth>
     <maxVel>1.0</maxVel>
-    <material>Gazebo/FlatBlack</material>
+    <material>Gazebo/Gold</material>
   </gazebo>
   <gazebo reference="imu_link">
@@ -54,5 +54,5 @@
       <visualize>$(arg imu_visual)</visualize>
     </sensor>
-    <material>Gazebo/Grey</material>
+    <material>Gazebo/Gold</material>
   </gazebo>
   <gazebo>

File: open_manipulator_with_tb3_description/urdf/turtlebot3_waffle_for_open_manipulator2.urdf.xacro (robot description, xacro)
@@ -30,6 +30,9 @@
       <origin xyz="0 0 0" rpy="0 0 0"/>
       <mass value="8.3729096e+0"/>
-      <inertia ixx="15.7002718e-03" ixy="-4.7576583e-05" ixz="1.1160499e-04"
+      <!--<inertia ixx="15.7002718e-03" ixy="-4.7576583e-05" ixz="1.1160499e-04"
                iyy="8.6195418e-03" iyz="-3.5422299e-06"
+               izz="1.4612727e-00" />-->
+      <inertia ixx="1.4612727e-00" ixy="-4.7576583e-05" ixz="1.1160499e-04"
+               iyy="1.4612727e-00" iyz="-3.5422299e-06"
                izz="1.4612727e-00" />
     </inertial>
