Commit message: add room3 modi

File: open_manipulator_with_tb3_description/urdf/turtlebot3_waffle_for_open_manipulator3.urdf.xacro (robot description, xacro)
@@ -29,15 +29,15 @@
     <inertial>
       <origin xyz="0 0 0" rpy="0 0 0"/>
-      <mass value="3.3729096e+0"/>
+      <mass value="8.3729096e+0"/>
       <!--<mass value="1.3729096e+00"/>-->
       <!--<inertia ixx="15.7002718e-03" ixy="-4.7576583e-05" ixz="1.1160499e-04"
                iyy="8.6195418e-03" iyz="-3.5422299e-06"
                izz="1.4612727e-00" />-->
-      <!--<inertia ixx="1.4612727e-00" ixy="-4.7576583e-05" ixz="1.1160499e-04"
+      <inertia ixx="1.4612727e-00" ixy="-4.7576583e-05" ixz="1.1160499e-04"
                iyy="1.4612727e-00" iyz="-3.5422299e-06"
-               izz="1.4612727e-00" />-->
-      <inertia ixx="8.7002718e-03" ixy="-4.7576583e-05" ixz="1.1160499e-04"
+               izz="1.4612727e-02" />
+      <!--<inertia ixx="8.7002718e-03" ixy="-4.7576583e-05" ixz="1.1160499e-04"
                iyy="8.6195418e-03" iyz="-3.5422299e-06"
-               izz="1.4612727e-02" />
+               izz="1.4612727e-02" />-->
     </inertial>
     <!--<inertial>
